File: PCB/LEMOAdaptorBoard6.kicad_pcb (KiCad board)
At the start: 2 copper layers, 52 x 107 mm, 15 parts

Commit message: update
Parts:
- added H5: MountingHole_3.2mm_M3, MountingHole_3.2mm_M3, F.Cu at (46.2, 25.3)
- added H6: MountingHole_3.2mm_M3, MountingHole_3.2mm_M3, F.Cu at (86.2, 25.3)
Other:
- board size 52 x 107 mm -> 52 x 117 mm
- board text added: "LEMOAdaptorBoard6 4CH FFC to LEMO BNC POWER INPUTS 2026-10-28"
- board text removed: "LEMOAdaptorBoard6 4CH FFC to LEMO BNC POWER INPUTS 2026-10-28, Au, Kei Yin Eltis"
Changed lines of the file:
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@@
 		(embedded_fonts no)
 	)
+	(footprint "MountingHole_3.2mm_M3"
+		(layer "F.Cu")
+		(at 46.16 25.28)
+		(descr "Mounting Hole 3.2mm, M3, no annular, generated by kicad-footprint-generator mountinghole.py")
+		(tags "mountinghole M3")
+		(property "Reference" "H5"
+			(at 0 -4.15 0)
+			(layer "F.SilkS")
+			(effects
+				(font
+					(size 1 1)
+					(thickness 0.15)
+				)
+			)
+		)
+		(property "Value" "MountingHole_3.2mm_M3"
+			(at 0 4.15 0)
+			(layer "F.Fab")
+			(effects
+				(font
+					(size 1 1)
+					(thickness 0.15)
+				)
+			)
+		)
+		(property "Datasheet" ""
+			(at 0 0 0)
+			(layer "F.Fab")
+			(hide yes)
+			(effects
+				(font
+					(size 1.27 1.27)
+					(thickness 0.15)
+				)
+			)
+		)
+		(property "Description" ""
+			(at 0 0 0)
+			(layer "F.Fab")
+			(hide yes)
+			(effects
+				(font
+					(size 1.27 1.27)
+					(thickness 0.15)
+				)
+			)
+		)
+		(attr board_only exclude_from_pos_files exclude_from_bom)
+		(fp_circle
+			(center 0 0)
+			(end 3.2 0)
+			(stroke
+				(width 0.15)
+				(type solid)
+			)
+			(fill no)
+			(layer "Cmts.User")
+		)
+		(fp_circle
+			(center 0 0)
+			(end 3.45 0)
+			(stroke
+				(width 0.05)
+				(type solid)
+			)
+			(fill no)
+			(layer "F.CrtYd")
+		)
+		(fp_text user "${REFERENCE}"
+			(at 0 0 0)
+			(layer "F.Fab")
+			(effects
+				(font
+					(size 1 1)
+					(thickness 0.15)
+				)
+			)
+		)
+		(pad "" np_thru_hole circle
+			(at 0 0)
+			(size 3.2 3.2)
+			(drill 3.2)
+			(layers "*.Cu" "*.Mask")
+		)
+		(embedded_fonts no)
+	)
 	(footprint "Board6:LEMO02"
 		(layer "F.Cu")
@@
 		(embedded_fonts no)
 	)
+	(footprint "MountingHole_3.2mm_M3"
+		(layer "F.Cu")
+		(at 86.16 25.28)
+		(descr "Mounting Hole 3.2mm, M3, no annular, generated by kicad-footprint-generator mountinghole.py")
+		(tags "mountinghole M3")
+		(property "Reference" "H6"
+			(at 0 -4.15 0)
+			(layer "F.SilkS")
+			(effects
+				(font
+					(size 1 1)
+					(thickness 0.15)
+				)
+			)
+		)
+		(property "Value" "MountingHole_3.2mm_M3"
+			(at 0 4.15 0)
+			(layer "F.Fab")
+			(effects
+				(font
+					(size 1 1)
+					(thickness 0.15)
+				)
+			)
+		)
+		(property "Datasheet" ""
+			(at 0 0 0)
+			(layer "F.Fab")
+			(hide yes)
+			(effects
+				(font
+					(size 1.27 1.27)
+					(thickness 0.15)
+				)
+			)
+		)
+		(property "Description" ""
+			(at 0 0 0)
+			(layer "F.Fab")
+			(hide yes)
+			(effects
+				(font
+					(size 1.27 1.27)
+					(thickness 0.15)
+				)
+			)
+		)
+		(attr board_only exclude_from_pos_files exclude_from_bom)
+		(fp_circle
+			(center 0 0)
+			(end 3.2 0)
+			(stroke
+				(width 0.15)
+				(type solid)
+			)
+			(fill no)
+			(layer "Cmts.User")
+		)
+		(fp_circle
+			(center 0 0)
+			(end 3.45 0)
+			(stroke
+				(width 0.05)
+				(type solid)
+			)
+			(fill no)
+			(layer "F.CrtYd")
+		)
+		(fp_text user "${REFERENCE}"
+			(at 0 0 0)
+			(layer "F.Fab")
+			(effects
+				(font
+					(size 1 1)
+					(thickness 0.15)
+				)
+			)
+		)
+		(pad "" np_thru_hole circle
+			(at 0 0)
+			(size 3.2 3.2)
+			(drill 3.2)
+			(layers "*.Cu" "*.Mask")
+		)
+		(embedded_fonts no)
+	)
 	(footprint "Board6:LEMO01"
 		(layer "F.Cu")
@@
 	)
 	(gr_rect
-		(start 40.16 29.28)
+		(start 40.16 19.28)
 		(end 92.16 136.28)
 		(stroke
@@
 		)
 	)
-	(gr_text "LEMOAdaptorBoard6\n4CH FFC to LEMO\nBNC POWER INPUTS\n2026-10-28,\nAu, Kei Yin Eltis"
+	(gr_text "LEMOAdaptorBoard6\n4CH FFC to LEMO\nBNC POWER INPUTS\n2026-10-28"
 		(at 70.66 104 90)
 		(layer "F.SilkS")
@@
 			(font
 				(size 1 1)
-				(thickness 0.25)
+				(thickness 0.3)
 				(bold yes)
 			)
@@
 		(polygon
 			(pts
-				(xy 41.16 30.28) (xy 41.16 135.28) (xy 91.16 135.28) (xy 91.16 30.28)
+				(xy 41.16 20.28) (xy 41.16 135.28) (xy 91.16 135.28) (xy 91.16 20.28)
 			)
 		)
